Commit message: Modification urdf v7

File: guardian_description/urdf/v7/guardian.urdf.xacro (robot description, xacro)
@@ -325,6 +325,15 @@
 	 <dynamics damping="100"/>
   </joint>
-  <link name="laser_tilt_mount_link">
-  </link>
+  <link name="laser_tilt_mount_link"></link>
+  <!--joint name="laser_tilt_mount_inverted_joint" type="fixed">
+     <axis xyz="0 1 0" />
+     <origin xyz="0 0 0" rpy="${PI} 0 0"/>
+     <parent link="laser_tilt_mount_link"/>
+     <child link="laser_tilt_mount_inverted_link"/>
+     <limit effort="30" lower="-2.6" upper="2.6" velocity="2.0"/>
+	 <dynamics damping="100"/>
+  </joint>
+  <link name="laser_tilt_mount_inverted_link">
+  </link-->
   <!-- HOKUYO FRONTAL ROTATION -->
   <joint name="laser_tilt_joint" type="revolute">

Commit message: changed guardian_tracks urdf descriptions
rviz_guardian_tracks.launch was duplicated

guardian tracks.urdf.xacro - commented out wheels; changed link and
joint names for more coherence with guardian.urdf; changed <robot> name

File: guardian_description/urdf/v7/guardian.urdf.xacro (robot description, xacro)
@@ -107,9 +107,9 @@
        <origin xyz="0 0 0" rpy="0 0 0" />
        <geometry>
-	 <mesh filename="package://guardian_description/meshes/others/v5/trackV5_l.dae"/>
-       </geometry>
-	<material name="black">
-		<color rgba="0.1 0.1 0.1 1"/>
-      	</material>
+	 	 <mesh filename="package://guardian_description/meshes/others/v5/trackV5_l.dae"/>
+       </geometry>
+	   <material name="black">
+		 <color rgba="0.1 0.1 0.1 1"/>
+       </material>
     </visual>
     <collision>
@@ -135,9 +135,9 @@
        <origin xyz="0 0 0" rpy="0 0 3.1416" />
        <geometry>
-	 <mesh filename="package://guardian_description/meshes/wheel.dae"/>
-       </geometry>
-	<material name="grey">
-		<color rgba="0.3 0.3 0.3 1"/>
-      	</material>
+	 	 <mesh filename="package://guardian_description/meshes/wheel.dae"/>
+       </geometry>
+	   <material name="grey">
+		 <color rgba="0.3 0.3 0.3 1"/>
+       </material>
     </visual>
     <collision>
@@ -178,7 +178,7 @@
          <mesh filename="package://guardian_description/meshes/wheel.dae"/>
        </geometry>
-	<material name="gray">
-		<color rgba="0.3 0.3 0.3 1"/>
-      	</material>
+	   <material name="gray">
+		 <color rgba="0.3 0.3 0.3 1"/>
+       </material>
     </visual>
     <collision>
@@ -219,7 +219,7 @@
          <mesh filename="package://guardian_description/meshes/wheel.dae"/>
        </geometry>
-	<material name="grey">
-		<color rgba="0.3 0.3 0.3 1"/>
-      	</material>
+	   <material name="grey">
+		 <color rgba="0.3 0.3 0.3 1"/>
+       </material>
     </visual>
     <collision>
@@ -260,7 +260,7 @@
          <mesh filename="package://guardian_description/meshes/wheel.dae"/>
        </geometry>
-	<material name="grey">
-		<color rgba="0.3 0.3 0.3 1"/>
-      	</material>
+	   <material name="grey">
+		 <color rgba="0.3 0.3 0.3 1"/>
+       </material>
     </visual>
     <collision>

File: guardian_description/urdf/v7/guardian_tracks.urdf.xacro (robot description, xacro)
@@ -1,4 +1,4 @@
 <?xml version="1.0"?>
-<robot name="gball" xmlns:xacro="http://www.ros.org/wiki/xacro">
+<robot name="guardian_tracks" xmlns:xacro="http://www.ros.org/wiki/xacro">
   <!-- Import all Gazebo-customization elements, including Gazebo colors -->
   <xacro:include filename="$(find guardian_description)/urdf/v7/guardian.gazebo" />
@@ -126,5 +126,5 @@
   </joint>
   <!-- BACK LEFT WHEEL (GREY) -->
-  <link name="back_left_wheel">
+  <!-- <link name="back_left_wheel">
     <inertial>
       <mass value="4.5" />
@@ -146,10 +146,10 @@
      <actuator name="joint_blw_motor">
 	    <hardwareInterface>EffortJointInterface</hardwareInterface>
-		<!-- hardwareInterface>VelocityJointInterface</hardwareInterface -->
+		hardwareInterface>VelocityJointInterface</hardwareInterface
         <mechanicalReduction>${wheel_mechanical_reduction}</mechanicalReduction>
-     	<!-- motorTorqueConstant>1</motorTorqueConstant -->
+     	motorTorqueConstant>1</motorTorqueConstant
      </actuator>
   </transmission>
-  <!-- BACK RIGHT WHEEL (BLACK) -->
+  BACK RIGHT WHEEL (BLACK)
   <link name="back_right_wheel">
     <inertial>
@@ -172,10 +172,10 @@
     <actuator name="joint_brw_motor">
 	   <hardwareInterface>EffortJointInterface</hardwareInterface>
-       <!-- hardwareInterface>VelocityJointInterface</hardwareInterface -->
+       hardwareInterface>VelocityJointInterface</hardwareInterface
        <mechanicalReduction>${wheel_mechanical_reduction}</mechanicalReduction>
-	   <!-- motorTorqueConstant>1</motorTorqueConstant -->
+	   motorTorqueConstant>1</motorTorqueConstant
     </actuator>
   </transmission>
-  <!-- FRONT LEFT WHEEL (GREY) -->
+  FRONT LEFT WHEEL (GREY)
   <link name="front_left_wheel">
     <inertial>
@@ -198,10 +198,10 @@
      <actuator name="joint_flw_motor">
 	   <hardwareInterface>EffortJointInterface</hardwareInterface>
-       <!-- hardwareInterface>VelocityJointInterface</hardwareInterface -->
+       hardwareInterface>VelocityJointInterface</hardwareInterface
        <mechanicalReduction>${wheel_mechanical_reduction}</mechanicalReduction>
-       <!-- motorTorqueConstant>1</motorTorqueConstant -->
+       motorTorqueConstant>1</motorTorqueConstant
      </actuator>
   </transmission>
-  <!-- FRONT RIGHT WHEEL (GREY) -->
+  FRONT RIGHT WHEEL (GREY)
   <link name="front_right_wheel">
     <inertial>
@@ -224,10 +224,11 @@
      <actuator name="joint_frw_motor">
 	   <hardwareInterface>EffortJointInterface</hardwareInterface>
-	   <!-- hardwareInterface>VelocityJointInterface</hardwareInterface -->
+	   hardwareInterface>VelocityJointInterface</hardwareInterface
        <mechanicalReduction>${wheel_mechanical_reduction}</mechanicalReduction>
-       <!-- motorTorqueConstant>1</motorTorqueConstant -->
+       motorTorqueConstant>1</motorTorqueConstant
      </actuator>
-     <!-- motorTorqueConstant>1</motorTorqueConstant -->
-  </transmission>
+     motorTorqueConstant>1</motorTorqueConstant
+  </transmission>
+ -->
   <!-- HOKUYO BACK SENSOR -->
   <joint name="hokuyo_back_laser_joint" type="fixed">
@@ -257,10 +258,29 @@
     </inertial>
   </link>
-  <!-- HOKUYO FRONTAL ROTATION -->
-  <joint name="hokuyo_frontal_laser_rotation_joint" type="revolute">
+  <joint name="laser_tilt_mount_joint" type="fixed">
      <axis xyz="0 1 0" />
      <origin xyz="0.46781 0 0.24299"/>
      <parent link="base_link"/>
-     <child link="hokuyo_frontal_laser_rotation_link"/>
+     <child link="laser_tilt_mount_link"/>
+     <limit effort="30" lower="-2.6" upper="2.6" velocity="2.0"/>
+	 <dynamics damping="100"/>
+  </joint>
+  <link name="laser_tilt_mount_link"></link>
+  <!--joint name="laser_tilt_mount_inverted_joint" type="fixed">
+     <axis xyz="0 1 0" />
+     <origin xyz="0 0 0" rpy="${PI} 0 0"/>
+     <parent link="laser_tilt_mount_link"/>
+     <child link="laser_tilt_mount_inverted_link"/>
+     <limit effort="30" lower="-2.6" upper="2.6" velocity="2.0"/>
+	 <dynamics damping="100"/>
+  </joint>
+  <link name="laser_tilt_mount_inverted_link">
+  </link-->
+  <!-- HOKUYO FRONTAL ROTATION -->
+  <joint name="laser_tilt_joint" type="revolute">
+     <axis xyz="0 1 0" />
+     <origin xyz="0 0 0"/>
+     <parent link="laser_tilt_mount_link"/>
+     <child link="laser_tilt_link"/>
      <limit effort="30" lower="-2.6" upper="2.6" velocity="2.0"/>
 	 <dynamics damping="100"/>
@@ -272,5 +292,5 @@
 	<motorTorqueConstant>1</motorTorqueConstant>
   </transmission>
-  <link name="hokuyo_frontal_laser_rotation_link">
+  <link name="laser_tilt_link">
      <visual>
        <origin xyz="0 0 0" rpy="0 0 0" />
@@ -295,5 +315,5 @@
      <axis xyz="0 1 0" />
      <origin xyz="0.066 0 0.0"/>
-     <parent link="hokuyo_frontal_laser_rotation_link"/>
+     <parent link="laser_tilt_link"/>
      <child link="hokuyo_frontal_laser_link"/>
   </joint>
