Commit message: guardian_description: setting sensor params and more

File: guardian_description/robots/v9/guardian_v9_wheels_all_sensors.urdf.xacro (robot description, xacro)
@@ -19,5 +19,5 @@
 	<xacro:guardian_wheels/>
 	<xacro:sensor_hokuyo_utm30lx name="hokuyo" parent="base_link">
-		<origin xyz="0.43171 0 0.29163" rpy="0 0 0"/>
+		<origin xyz="0.44171 0 0.31163" rpy="0 0 0"/>
 	</xacro:sensor_hokuyo_utm30lx>
 	<xacro:sensor_imu name="imu" parent="base_link">
@@ -32,4 +32,4 @@
 	<xacro:gazebo_guardian_skid_steering broadcastOdomTF="1" namespace="/guardian"/>
 	<!-- Gazebo ros control pluggins -->
-	<xacro:ros_control namespace="/guardian"/>
+	<xacro:ros_control_guardian namespace="/guardian"/>
 </robot>

File: guardian_description/urdf/sensors/hokuyo_utm30lx.urdf.xacro (robot description, xacro)
@@ -40,6 +40,6 @@
 							<samples>1081</samples>
 							<resolution>1</resolution>
-							<min_angle>2.35619449</min_angle>  <!-- +/-135 deg -->
-							<max_angle>-2.35619449</max_angle>
+							<min_angle>2.09</min_angle>  <!-- +/-120 deg -->
+							<max_angle>-2.09</max_angle>
 						</horizontal>
 					</scan>

File: guardian_description/urdf/sensors/kinect.urdf.xacro (robot description, xacro)
@@ -107,4 +107,9 @@
             <far>8.0</far>
           </clip>
+	  <noise>
+	  	<type>gaussian</type>
+		<mean>0.0</mean>
+		<stddev>0.07</stddev>
+	  </noise>
         </camera>
         <plugin name="kinect_cam_controller" filename="libgazebo_ros_openni_kinect.so">

File: guardian_description/urdf/v9/guardian.gazebo.xacro (robot description, xacro)
@@ -2,5 +2,5 @@
 <robot xmlns:xacro="http://ros.org/wiki/xacro">
   <!-- ros_control plugin -->
-  <xacro:macro name="ros_control" params="namespace">
+  <xacro:macro name="ros_control_guardian" params="namespace">
 	  <gazebo>
 		<plugin name="ros_control" filename="libgazebo_ros_control.so">
