Commit message: Minor changes

File: guardian_description/urdf/guardian.urdf.xacro (robot description, xacro)
@@ -18,10 +18,4 @@
   <xacro:property name="ptz_joint_damping" value="0.1" />
   <xacro:property name="ptz_mechanical_reduction" value="1.0" />
-  <!-- Used for fixing robot to Gazebo 'base_link' -->
-  <!-- link name="world"/>
-  <joint name="fwf" type="planar">
-    <parent link="world"/>
-    <child link="base_footprint"/>
-  </joint -->
   <!-- BASE FOOTPRINT -->
   <!-- base_footprint is a fictitious link(frame) that is on the ground right below base_link origin,
@@ -59,5 +53,6 @@
        <origin xyz="0 0 0" rpy="0 0 0" />
        <geometry>
-	 <mesh filename="package://guardian_description/meshes/chassis/v6/chassisV6.dae"/>
+	 <mesh filename="package://guardian_description/meshes/chassis/v5/chassisV5_1.stl"/>
+	 <!--mesh filename="package://guardian_description/meshes/chassis/v6/chassisV6.dae"/-->
        </geometry>
     </visual>
@@ -65,5 +60,5 @@
        <origin xyz="0 0 0" rpy="0 0 0 " />
        <geometry>
-         <mesh filename="package://guardian_description/meshes/chassis/v6/chassisV6.dae"/>
+         <mesh filename="package://guardian_description/meshes/chassis/v5/chassisV5_1.stl"/>
        </geometry>
     </collision>
@@ -299,5 +294,5 @@
   </transmission>
 	<!-- KINECT CAMERA -->
-  <joint name="camera_joint" type="fixed">
+  <!--joint name="camera_joint" type="fixed">
      <axis xyz="0 1 0" />
      <origin xyz="0.5 0 0.31"/>
@@ -311,7 +306,7 @@
        <inertia ixx="0.0001" ixy="0" ixz="0" iyy="0.000001" iyz="0" izz="0.0001" />
     </inertial>
-  </link>
+  </link-->
   <!-- HOKUYO REAR SENSOR -->
-  <joint name="hokuyo_laser_joint" type="fixed">
+  <!--joint name="hokuyo_laser_joint" type="fixed">
      <axis xyz="0 1 0" />
      <origin xyz="-0.43171 0 0.29163"/>
@@ -319,5 +314,4 @@
      <child link="hokuyo_laser_link"/>
   </joint>
-  <!-- Hokuyo Laser -->
   <link name="hokuyo_laser_link">
     <collision>
@@ -327,10 +321,4 @@
       </geometry>
     </collision>
-    <!-- visual>
-      <origin xyz="0 0 0" rpy="0 0 0"/>
-      <geometry>
-        <mesh filename="package://guardian_description/meshes/hokuyo-utm30-lx.dae"/>
-      </geometry>
-    </visual -->
     <inertial>
       <mass value="1e-5" />
@@ -338,5 +326,5 @@
       <inertia ixx="1e-6" ixy="0" ixz="0" iyy="1e-6" iyz="0" izz="1e-6" />
     </inertial>
-  </link>
+  </link-->
   <!-- IMU SENSOR -->
   <joint name="imu_joint" type="fixed">
@@ -366,5 +354,5 @@
   </link>
   <!-- AXIS PTZ CAMERA WITH PAN AND TILT -->
-  <link name="camera_base_link">
+  <!--link name="camera_base_link">
      <inertial>
        <mass value="0.1" />
@@ -424,4 +412,4 @@
        <mechanicalReduction>${ptz_mechanical_reduction}</mechanicalReduction>
      </actuator>
-  </transmission>
+  </transmission -->
 </robot>
